File: Hardware/v0/ergonomic_split_left/USB_UPSTREAM.sch (KiCad schematic (older format))
At the start: 14 parts, among them J1 USB_C_Receptacle_USB2.0, U2 SRV05-4

Commit message: Connecting schematic blocks, most sub-blocks done
Connections:
- net +5V0_USB renamed +5V
- net USB_UPSTREAM_OUT+ renamed USB+
- net USB_UPSTREAM_OUT- renamed USB-
Other:
- moved on the sheet: C1, C2, C3, FB1, FB2, FB3, J1, L1, R1, R2, R42, R5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

Commit message: Debug connectors Adding I2C debug header Changed SPI programming header to edge mount Changed right interface connector to IDC Cleaning up schematic
Parts:
- removed R42: 1K5, resistor_smd:R_0603_1608Metric, symbol Device:R
Changed lines of the file:
@@
 Wire Wire Line
 	6200 3475 6525 3475
-Wire Wire Line
-	6925 3475 7025 3475
 Connection ~ 6225 2375
 Wire Wire Line
@@
 Wire Wire Line
 	7575 4525 7725 4525
-$Comp
-L Device:R R?
-U 1 1 614B1649
-P 7025 2975
-AR Path="/6114D32E/614B1649" Ref="R?"  Part="1"
-AR Path="/6247A5CE/614B1649" Ref="R?"  Part="1"
-AR Path="/612340DE/614B1649" Ref="R?"  Part="1"
-AR Path="/62F6B81F/614B1649" Ref="R42"  Part="1"
-AR Path="/629982B4/614B1649" Ref="R42"  Part="1"
-F 0 "R42" V 6950 2975 50  0000 C CNN
-F 1 "1K5" V 7025 2975 50  0000 C CNN
-F 2 "resistor_smd:R_0603_1608Metric" V 6955 2975 50  0001 C CNN
-F 3 "~" H 7025 2975 50  0001 C CNN
-	1    7025 2975
-	1    0    0    1
-$EndComp
-Wire Wire Line
-	7025 3125 7025 3475
-Connection ~ 7025 3475
-Wire Wire Line
-	7025 3475 7250 3475
-$Comp
-L power:+3.3V #PWR?
-U 1 1 614B6C4F
-P 7025 2775
-AR Path="/6114D32E/614B6C4F" Ref="#PWR?"  Part="1"
-AR Path="/6247A5CE/614B6C4F" Ref="#PWR?"  Part="1"
-AR Path="/612340DE/614B6C4F" Ref="#PWR?"  Part="1"
-AR Path="/62F6B81F/614B6C4F" Ref="#PWR0538"  Part="1"
-AR Path="/613390DE/614B6C4F" Ref="#PWR?"  Part="1"
-AR Path="/629982B4/614B6C4F" Ref="#PWR0538"  Part="1"
-F 0 "#PWR0538" H 7025 2625 50  0001 C CNN
-F 1 "+3.3V" H 7040 2948 50  0000 C CNN
-F 2 "" H 7025 2775 50  0001 C CNN
-F 3 "" H 7025 2775 50  0001 C CNN
-	1    7025 2775
-	1    0    0    -1
-$EndComp
-Wire Wire Line
-	7025 2825 7025 2775
 $Comp
 L power:+5V #PWR011
@@
 	1    0    0    -1
 $EndComp
+Wire Wire Line
+	6925 3475 7250 3475
 $EndSCHEMATC

Commit message: Prelim routing done
Connections:
- net CD+: now also U2.4 (IO3); no longer U2.3 (IO2)
- net CD-: now also U2.3 (IO2); no longer U2.4 (IO3)
Changed lines of the file:
@@
 	-1   0    0    -1
 $EndComp
-Wire Wire Line
-	6325 3275 6325 3800
 NoConn ~ 7575 4725
 Wire Wire Line
@@
 Text Notes 6325 3950 0    50   ~ 0
 ESD Protection
-Wire Wire Line
-	6325 3800 7725 3800
-Wire Wire Line
-	7725 3800 7725 4525
 NoConn ~ 6575 4525
 Wire Wire Line
@@
 Wire Wire Line
 	5400 3275 6325 3275
-Wire Wire Line
-	5400 3475 6200 3475
 Connection ~ 6325 3275
-Connection ~ 6200 3475
 Text Label 5775 3275 0    50   ~ 0
 CD-
@@
 Wire Wire Line
 	6925 3275 7250 3275
-Wire Wire Line
-	6200 3475 6525 3475
 Connection ~ 6225 2375
-Wire Wire Line
-	6200 4725 6575 4725
-Wire Wire Line
-	6200 3475 6200 4725
-Wire Wire Line
-	7575 4525 7725 4525
 $Comp
 L power:+5V #PWR011
@@
 Wire Wire Line
 	6925 3475 7250 3475
+Wire Wire Line
+	5400 3475 6425 3475
+Wire Wire Line
+	6325 4725 6575 4725
+Wire Wire Line
+	6325 3275 6325 4725
+Wire Wire Line
+	6425 3475 6425 3750
+Wire Wire Line
+	6425 3750 7700 3750
+Wire Wire Line
+	7700 3750 7700 4525
+Wire Wire Line
+	7700 4525 7575 4525
+Connection ~ 6425 3475
+Wire Wire Line
+	6425 3475 6525 3475
 $EndSCHEMATC
