File: Hardware/v0/ergonomic_split_left/ergonomic_split_left.kicad_pcb (KiCad board)
At the start: 2 copper layers, 105 parts, among them J1 USB_C_Receptacle_USB2.0, J5 Conn_02x03_Odd_Even, SW1 SW_Push, SW100 L41, SW101 L51, SW102 L02, SW103 L12, SW104 L22, SW105 L32, SW106 L42, SW107 L52, SW108 L03, SW109 L13, SW110 L23, SW111 L33, SW112 L43, SW114 L04, SW115 L14, SW116 L24, SW117 L34, SW118 L44, SW119 L54, SW120 L05, SW121 L15, SW122 L25, SW123 L25, SW124 L55, SW125 L06, SW126 L16, SW127 L36, SW128 L56, SW90 L00, SW91 L10, SW92 L20, SW94 L30, SW95 L40, SW96 L01, SW97 L11, SW98 L21, SW99 L31, U1 SRV05-4, U6 ATmega32U4-AU, X2 KC2016K

Commit message: Switch matrix placement
Parts:
- removed D1, D10, D11, D12, D120, D121, D122, D123, D124, D125, D126, D13, D14, D15, D16, D17, D18, D19, D2, D20, D21, D22, D23, D24, D25, D26, D27, D28, D29, D3, D30, D31, D4, D5, D6, D7, D8, D9: D, custom_footprint_library:SOD323_HS
- removed SW100: L41, CherryMX_PCB_KailhSocket:CherryMX_1.00u_PCB_KailhSocket
- removed SW101: L51, CherryMX_PCB_KailhSocket:CherryMX_1.00u_PCB_KailhSocket
- removed SW102: L02, CherryMX_PCB_KailhSocket:CherryMX_1.00u_PCB_KailhSocket
- removed SW103: L12, CherryMX_PCB_KailhSocket:CherryMX_1.00u_PCB_KailhSocket
- removed SW104: L22, CherryMX_PCB_KailhSocket:CherryMX_1.00u_PCB_KailhSocket
- removed SW105: L32, CherryMX_PCB_KailhSocket:CherryMX_1.00u_PCB_KailhSocket
- removed SW106: L42, CherryMX_PCB_KailhSocket:CherryMX_1.00u_PCB_KailhSocket
- removed SW107: L52, CherryMX_PCB_KailhSocket:CherryMX_2.00u_PCB_KailhSocket
- removed SW108: L03, CherryMX_PCB_KailhSocket:CherryMX_1.00u_PCB_KailhSocket
- removed SW109: L13, CherryMX_PCB_KailhSocket:CherryMX_1.00u_PCB_KailhSocket
- removed SW110: L23, CherryMX_PCB_KailhSocket:CherryMX_1.00u_PCB_KailhSocket
- removed SW111: L33, CherryMX_PCB_KailhSocket:CherryMX_1.00u_PCB_KailhSocket
- removed SW112: L43, CherryMX_PCB_KailhSocket:CherryMX_1.00u_PCB_KailhSocket
- removed SW114: L04, CherryMX_PCB_KailhSocket:CherryMX_1.00u_PCB_KailhSocket
- removed SW115: L14, CherryMX_PCB_KailhSocket:CherryMX_1.00u_PCB_KailhSocket
- removed SW116: L24, CherryMX_PCB_KailhSocket:CherryMX_1.00u_PCB_KailhSocket
- removed SW117: L34, CherryMX_PCB_KailhSocket:CherryMX_1.00u_PCB_KailhSocket
- removed SW118: L44, CherryMX_PCB_KailhSocket:CherryMX_1.00u_PCB_KailhSocket
- removed SW119: L54, CherryMX_PCB_KailhSocket:CherryMX_1.00u_PCB_KailhSocket
- removed SW120: L05, CherryMX_PCB_KailhSocket:CherryMX_1.00u_PCB_KailhSocket
- removed SW121: L15, CherryMX_PCB_KailhSocket:CherryMX_1.00u_PCB_KailhSocket
- removed SW122, SW123: L25, CherryMX_PCB_KailhSocket:CherryMX_1.00u_PCB_KailhSocket
- removed SW124: L55, CherryMX_PCB_KailhSocket:CherryMX_1.00u_PCB_KailhSocket
- removed SW125: L06, CherryMX_PCB_KailhSocket:CherryMX_1.00u_PCB_KailhSocket
- removed SW126: L16, CherryMX_PCB_KailhSocket:CherryMX_1.50u_PCB_KailhSocket
- removed SW127: L36, CherryMX_PCB_KailhSocket:CherryMX_1.50u_PCB_KailhSocket
- removed SW128: L56, CherryMX_PCB_KailhSocket:CherryMX_1.00u_PCB_KailhSocket
- removed SW90: L00, CherryMX_PCB_KailhSocket:CherryMX_1.50u_PCB_KailhSocket
- removed SW91: L10, CherryMX_PCB_KailhSocket:CherryMX_1.50u_PCB_KailhSocket
- removed SW92: L20, CherryMX_PCB_KailhSocket:CherryMX_1.50u_PCB_KailhSocket
- removed SW94: L30, CherryMX_PCB_KailhSocket:CherryMX_1.50u_PCB_KailhSocket
- removed SW95: L40, CherryMX_PCB_KailhSocket:CherryMX_1.50u_PCB_KailhSocket
- removed SW96: L01, CherryMX_PCB_KailhSocket:CherryMX_1.00u_PCB_KailhSocket
- removed SW97: L11, CherryMX_PCB_KailhSocket:CherryMX_1.00u_PCB_KailhSocket
- removed SW98: L21, CherryMX_PCB_KailhSocket:CherryMX_1.00u_PCB_KailhSocket
- removed SW99: L31, CherryMX_PCB_KailhSocket:CherryMX_1.00u_PCB_KailhSocket
- removed SWE: L53, CherryMX_PCB_KailhSocket:CherryMX_2.00u_PCB_KailhSocket
- added SW10: L31, custom_footprint_library:CherryMX_1.00u_KailhSocket_Integrated_Reversed, F.Cu at (94.5, 109.5)
- added SW11: L41, custom_footprint_library:CherryMX_1.00u_KailhSocket_Integrated, F.Cu at (94.5, 128.6)
- added SW12: L51, custom_footprint_library:CherryMX_1.00u_KailhSocket_Integrated, F.Cu at (193.7, 173.8)
- added SW13: L02, custom_footprint_library:CherryMX_1.00u_KailhSocket_Integrated, F.Cu at (113.5, 50.0)
- added SW14: L12, custom_footprint_library:CherryMX_1.00u_KailhSocket_Integrated_Reversed, F.Cu at (113.5, 69.1)
- added SW15: L22, custom_footprint_library:CherryMX_1.00u_KailhSocket_Integrated, F.Cu at (113.5, 88.1)
- added SW16: L32, custom_footprint_library:CherryMX_1.00u_KailhSocket_Integrated_Reversed, F.Cu at (113.5, 107.2)
- added SW17: L42, custom_footprint_library:CherryMX_1.00u_KailhSocket_Integrated, F.Cu at (113.5, 126.2)
- added SW18: L52, custom_footprint_library:CherryMX_2.00u_KailhSocket_Integrated_Vertical, F.Cu at (186.8, 153.6)
- added SW19: L03, custom_footprint_library:CherryMX_1.00u_KailhSocket_Integrated, F.Cu at (132.6, 47.6)
- added SW2: L00, custom_footprint_library:CherryMX_1.50u_KailhSocket_Integrated, F.Cu at (70.6, 52.4)
- added SW20: L13, custom_footprint_library:CherryMX_1.00u_KailhSocket_Integrated_Reversed, F.Cu at (132.6, 66.7)
- added SW21: L23, custom_footprint_library:CherryMX_1.00u_KailhSocket_Integrated, F.Cu at (132.6, 85.7)
- added SW22: L33, custom_footprint_library:CherryMX_1.00u_KailhSocket_Integrated_Reversed, F.Cu at (132.6, 104.8)
- added SW23: L43, custom_footprint_library:CherryMX_1.00u_KailhSocket_Integrated, F.Cu at (132.6, 123.8)
- added SW24: L53, custom_footprint_library:CherryMX_2.00u_KailhSocket_Integrated_Vertical, F.Cu at (173.3, 140.1)
- added SW25: L04, custom_footprint_library:CherryMX_1.00u_KailhSocket_Integrated, F.Cu at (151.6, 50.0)
- added SW26: L14, custom_footprint_library:CherryMX_1.00u_KailhSocket_Integrated_Reversed, F.Cu at (151.6, 69.1)
- added SW27: L24, custom_footprint_library:CherryMX_1.00u_KailhSocket_Integrated, F.Cu at (151.6, 88.1)
- added SW28: L34, custom_footprint_library:CherryMX_1.00u_KailhSocket_Integrated_Reversed, F.Cu at (151.6, 107.2)
- added SW29: L44, custom_footprint_library:CherryMX_1.00u_KailhSocket_Integrated, F.Cu at (151.6, 126.2)
- added SW3: L10, custom_footprint_library:CherryMX_1.50u_KailhSocket_Integrated_Reversed, F.Cu at (70.6, 71.4)
- added SW30: L54, custom_footprint_library:CherryMX_1.00u_KailhSocket_Integrated_Reversed, F.Cu at (207.2, 160.3)
- added SW31: L05, custom_footprint_library:CherryMX_1.00u_KailhSocket_Integrated, F.Cu at (170.7, 52.4)
- added SW32: L15, custom_footprint_library:CherryMX_1.00u_KailhSocket_Integrated_Reversed, F.Cu at (170.7, 71.4)
- added SW33: L25, custom_footprint_library:CherryMX_1.00u_KailhSocket_Integrated, F.Cu at (170.7, 90.5)
- added SW34: L35, custom_footprint_library:CherryMX_1.00u_KailhSocket_Integrated_Reversed, F.Cu at (170.7, 109.5)
- added SW35: L55, custom_footprint_library:CherryMX_1.00u_KailhSocket_Integrated_Reversed, F.Cu at (207.2, 133.3)
- added SW36: L16, custom_footprint_library:CherryMX_1.50u_KailhSocket_Integrated_Vertical_Reversed, F.Cu at (189.7, 76.2)
- added SW37: L36, custom_footprint_library:CherryMX_1.50u_KailhSocket_Integrated_Vertical_Reversed, F.Cu at (189.7, 104.8)
- added SW38: L56, custom_footprint_library:CherryMX_1.00u_KailhSocket_Integrated_Reversed, F.Cu at (220.7, 146.8)
- added SW39: L06, custom_footprint_library:CherryMX_1.00u_KailhSocket_Integrated, F.Cu at (189.7, 52.4)
- added SW4: L20, custom_footprint_library:CherryMX_1.50u_KailhSocket_Integrated, F.Cu at (70.6, 90.5)
- added SW5: L30, custom_footprint_library:CherryMX_1.50u_KailhSocket_Integrated_Reversed, F.Cu at (70.6, 109.5)
- added SW6: L40, custom_footprint_library:CherryMX_1.50u_KailhSocket_Integrated, F.Cu at (70.6, 128.6)
- added SW7: L01, custom_footprint_library:CherryMX_1.00u_KailhSocket_Integrated, F.Cu at (94.5, 52.4)
- added SW8: L11, custom_footprint_library:CherryMX_1.00u_KailhSocket_Integrated_Reversed, F.Cu at (94.5, 71.4)
- added SW9: L21, custom_footprint_library:CherryMX_1.00u_KailhSocket_Integrated, F.Cu at (94.5, 90.5)
- moved C1 136.9 mm to (740.8, 99.9)
- moved R1 136.9 mm to (732.6, 107.3)
- moved R22 136.9 mm to (541.2, 221.3)
- moved TP2 136.9 mm to (542.2, 224.1)
- moved U6 136.9 mm to (525.4, 217.2)
- moved C2 136.9 mm to (720.6, 108.4)
- moved C3 136.9 mm to (736.7, 106.8)
- moved C42 136.9 mm to (538.6, 224.1)
- moved C43 136.9 mm to (541.2, 218.8)
- moved C44 136.9 mm to (541.2, 216.3)
- moved C45 136.9 mm to (540.7, 213.8)
- moved C46 136.9 mm to (544.7, 211.2)
- moved FB1 136.9 mm to (732.5, 104.7)
- moved FB3 136.9 mm to (732.5, 101.9)
- moved J1 136.9 mm to (721.4, 97.5)
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Other:
- board outline added: 4.5 x 4.5 mm

Commit message: Connecting schematic blocks, most sub-blocks done
Parts:
- added C120: 1uF, Capacitor_smd:C_0603_1608Metric, F.Cu at (377.5, 73.9)
- added C4: 100nF, Capacitor_smd:C_0603_1608Metric, F.Cu at (262.7, 46.8)
- added C5: 100nF, Capacitor_smd:C_0603_1608Metric, F.Cu at (377.5, 71.4)
- added C6: 100nF, Capacitor_smd:C_0603_1608Metric, F.Cu at (262.7, 49.3)
- added R10: 1K, resistor_smd:R_0603_1608Metric, F.Cu at (266.7, 51.9)
- added R11: 10K, resistor_smd:R_0603_1608Metric, F.Cu at (146.1, 58.7)
- added R12: 10K, resistor_smd:R_0603_1608Metric, F.Cu at (146.1, 61.2)
- added R13: 10K, resistor_smd:R_0603_1608Metric, F.Cu at (150.1, 58.7)
- added R14: 2K2, resistor_smd:R_0603_1608Metric, F.Cu at (356.4, 124.6)
- added R15: 2K2, resistor_smd:R_0603_1608Metric, F.Cu at (360.4, 124.6)
- added R4: 10K, resistor_smd:R_0603_1608Metric, F.Cu at (266.7, 46.8)
- added R7: 10K, resistor_smd:R_0603_1608Metric, F.Cu at (262.7, 51.9)
- added R8: 1K, resistor_smd:R_0603_1608Metric, F.Cu at (266.7, 49.3)
- added R9: 1K, resistor_smd:R_0603_1608Metric, F.Cu at (262.7, 54.4)
- added SW40: L_Encoder, Rotary_Encoder:RotaryEncoder_Alps_EC11E-Switch_Vertical_H20mm, F.Cu at (211.9, 31.0)
- added U2: PCAL9555AHF, custom_footprint_library:QFN-24_EP_5x5_Pitch0.5mm, F.Cu at (153.5, 66.1)
- added U9: TCR2EF33, custom_footprint_library:TCR2EF33_SOT25, F.Cu at (372.4, 73.6)
- SW10, SW14, SW16, SW20, SW22, SW26, SW28, SW30, SW32, SW34, SW35, SW38, SW8: footprint custom_footprint_library:CherryMX_1.00u_KailhSocket_Integrated_Reversed -> custom_footprint_library:CherryMX_1.00u_KailhSocket_Integrated
- SW11, SW12, SW13, SW15, SW17, SW19, SW21, SW23, SW25, SW27, SW29, SW31, SW33, SW39, SW7, SW9: footprint custom_footprint_library:CherryMX_1.00u_KailhSocket_Integrated -> custom_footprint_library:CherryMX_1.00u_KailhSocket_Integrated_Reversed
- SW18, SW24: footprint custom_footprint_library:CherryMX_2.00u_KailhSocket_Integrated_Vertical -> custom_footprint_library:CherryMX_2.00u_KailhSocket_Integrated_Vertical_Reversed
- SW2, SW4, SW6: footprint custom_footprint_library:CherryMX_1.50u_KailhSocket_Integrated -> custom_footprint_library:CherryMX_1.50u_KailhSocket_Integrated_Reversed
- SW3, SW5: footprint custom_footprint_library:CherryMX_1.50u_KailhSocket_Integrated_Reversed -> custom_footprint_library:CherryMX_1.50u_KailhSocket_Integrated
- SW36, SW37: footprint custom_footprint_library:CherryMX_1.50u_KailhSocket_Integrated_Vertical_Reversed -> custom_footprint_library:CherryMX_1.50u_KailhSocket_Integrated_Vertical
- moved C1 369.0 mm to (377.2, 36.4)
- moved R1 369.0 mm to (369.1, 43.8)
- moved FB2 369.0 mm to (373.8, 33.8)
- moved J1 369.0 mm to (357.9, 34.0)
- moved C2 369.0 mm to (357.1, 44.9)
- moved C3 369.0 mm to (373.2, 43.3)
- moved FB1 369.0 mm to (368.9, 41.2)
- moved FB3 369.0 mm to (368.9, 38.4)
- moved L1 369.0 mm to (376.5, 39.4)
- moved R2 369.0 mm to (373.2, 40.8)
- moved R42 369.0 mm to (373.2, 38.3)
- moved R5 369.0 mm to (365.1, 44.9)
- moved R6 369.0 mm to (361.1, 44.9)
- moved U1 369.0 mm to (369.1, 34.7)
- moved U6 183.3 mm to (361.9, 134.1), turned to 180 degrees
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Connections:
- net /Switch Matrix/COL[0] renamed /IO Expander/COL[0]
- net /Switch Matrix/COL[1] renamed /IO Expander/COL[1]
- net /Switch Matrix/COL[2] renamed /IO Expander/COL[2]
- net /Switch Matrix/COL[3] renamed /IO Expander/COL[3]
- net /Switch Matrix/COL[4] renamed /IO Expander/COL[4]
- net /Switch Matrix/COL[5] renamed /IO Expander/COL[5]
- net /Switch Matrix/COL[6] renamed /IO Expander/COL[6]
- net /Switch Matrix/ROW[0] renamed /IO Expander/ROW[0]
- net /Switch Matrix/ROW[1] renamed /IO Expander/ROW[1]
- net /Switch Matrix/ROW[2] renamed /IO Expander/ROW[2]
- net /Switch Matrix/ROW[3] renamed /IO Expander/ROW[3]
- net /Switch Matrix/ROW[4] renamed /IO Expander/ROW[4]
- net /Switch Matrix/ROW[5] renamed /IO Expander/ROW[5]
- net MISO renamed /uController/MISO
- net MOSI renamed /uController/MOSI
- net Net-(U6-Pad38) renamed /uController/ENCODER_B_R
- net Net-(U6-Pad39) renamed /uController/ENCODER_A_R
- net Net-(U6-Pad40) renamed /uController/ENCODER_SW_R
- net RST renamed /uController/RST
- net SCK renamed /uController/SCK
- C3 pad 1: +5V0_USB -> +5V
- FB3 pad 1: +5V0_USB -> +5V
- R3 pad 1: nCAPS -> /uController/nCAPS_LED
- R5 pad 1: /USB_UPSTREAM/USB_UPSTREAM_OUT- -> /USB_UPSTREAM/USB-
- R6 pad 1: /USB_UPSTREAM/USB_UPSTREAM_OUT+ -> /USB_UPSTREAM/USB+
- U6 pad 18: /uController/SCL -> /IO Expander/SCL
- U6 pad 19: /uController/SDA -> /IO Expander/SDA
- U6 pad 22: Net-(U6-Pad22) -> /uController/nCAPS_LED
- U6 pad 25: Net-(U6-Pad25) -> /Switch Matrix/ENCODER_SW_L
- U6 pad 26: Net-(U6-Pad26) -> /Switch Matrix/ENCODER_A_L
- U6 pad 27: Net-(U6-Pad27) -> /Switch Matrix/ENCODER_B_L
- U6 pad 3: /uController/USB_IN- -> /USB_UPSTREAM/USB-
- U6 pad 30: /uController/RGB_DOUT -> /Switch Matrix/RGB_DIN
- U6 pad 4: /uController/USB_IN+ -> /USB_UPSTREAM/USB+

Commit message: Drawing board outline Basic placement done Adding rotary encoder to the switch matrix Adding mounting holes
Parts:
- removed R10: 1K, resistor_smd:R_0603_1608Metric
- added C7: 100nF, Capacitor_smd:C_0603_1608Metric, F.Cu at (111.0, 65.9)
- added D1: D, custom_footprint_library:SOD323_HS, B.Cu at (181.7, 76.5)
- added H1: MountingHole_Pad, mounting_hole:MountingHole_3.2mm_M3_ISO7380_Pad, F.Cu at (76.2, 58.8)
- added H10: MountingHole_Pad, mounting_hole:MountingHole_3.2mm_M3_ISO7380_Pad, F.Cu at (216.7, 160.7)
- added H2: MountingHole_Pad, mounting_hole:MountingHole_3.2mm_M3_ISO7380_Pad, F.Cu at (76.2, 177.9)
- added H3: MountingHole_Pad, mounting_hole:MountingHole_3.2mm_M3_ISO7380_Pad, F.Cu at (216.7, 225.7)
- added H4: MountingHole_Pad, mounting_hole:MountingHole_3.2mm_M3_ISO7380_Pad, F.Cu at (105.6, 137.7)
- added H5: MountingHole_Pad, mounting_hole:MountingHole_3.2mm_M3_ISO7380_Pad, F.Cu at (146.5, 58.8)
- added H6: MountingHole_Pad, mounting_hole:MountingHole_3.2mm_M3_ISO7380_Pad, F.Cu at (259.1, 183.4)
- added H7: MountingHole_Pad, mounting_hole:MountingHole_3.2mm_M3_ISO7380_Pad, F.Cu at (105.4, 98.8)
- added H8: MountingHole_Pad, mounting_hole:MountingHole_3.2mm_M3_ISO7380_Pad, F.Cu at (225.5, 58.8)
- added H9: MountingHole_Pad, mounting_hole:MountingHole_3.2mm_M3_ISO7380_Pad, F.Cu at (216.9, 101.6)
- C4, C6, R4, R7, R8, R9, TP2, U1: moved to B.Cu
- moved R3 305.0 mm to (90.4, 61.5), turned to 180 degrees
- moved D194 301.0 mm to (90.3, 60.0)
- moved TP2 298.4 mm to (95.6, 69.5)
- moved C44 275.6 mm to (118.0, 63.5)
- moved X2 271.2 mm to (127.7, 60.4), turned to 90 degrees
- moved C42 269.2 mm to (127.3, 58.2), turned to 180 degrees
- moved R23 268.6 mm to (118.2, 73.1), turned to 180 degrees
- moved C46 258.1 mm to (137.4, 66.0)
- moved C43 257.0 mm to (136.8, 68.8)
- moved R22 256.1 mm to (149.7, 43.4), turned to 225 degrees
- moved C45 253.5 mm to (136.3, 74.6)
- moved J5 252.9 mm to (144.0, 38.9), turned to 45 degrees
- moved SW1 249.1 mm to (153.9, 39.8), turned to 90 degrees
- moved R15 248.4 mm to (121.1, 57.9)
- moved R14 243.8 mm to (121.5, 59.3)
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Connections:
- net /Switch Matrix/RGB_DOUT renamed /Right Interface/RGB_DIN
- net /uController/ENCODER_A_R renamed /Right Interface/ENCODER_A_R
- net /uController/ENCODER_B_R renamed /Right Interface/ENCODER_B_R
- net /uController/ENCODER_SW_R renamed Net-(U6-Pad40)
- SW40 pad S1: +3V3 -> Net-(D1-Pad2)
- SW40 pad S2: /Switch Matrix/ENCODER_SW_L -> /IO Expander/COL[6]
- U2 pad 7: Net-(U2-Pad7) -> /IO Expander/ROW[6]
- U6 pad 25: /Switch Matrix/ENCODER_SW_L -> Net-(U6-Pad25)
Other:
- board size 4.5 x 4.5 mm -> 189.3 x 173.4 mm
