File: Hardware/v0/ergonomic_split_left/ergonomic_split_left.kicad_pcb (KiCad board)
At the start: 2 copper layers, 182.6 x 172.4 mm, 96 parts, among them J1 USB_C_Receptacle_USB2.0, J2 Right_Interface, J3 Conn_01x02_Male, J5 Conn_02x03_Odd_Even, SW1 SW_Push, SW10 L31, SW11 L41, SW12 L51, SW13 L02, SW14 L12, SW15 L22, SW16 L32, SW17 L42, SW18 L52, SW19 L03, SW2 L00, SW20 L13, SW21 L23, SW22 L33, SW23 L43, SW24 L53, SW25 L04, SW26 L14, SW27 L24, SW28 L34, SW29 L44, SW3 L10, SW30 L54, SW31 L05, SW32 L15, SW33 L25, SW34 L35, SW35 L55, SW36 L16, SW37 L36, SW38 L56, SW39 L06, SW4 L20, SW40 L_Encoder, SW5 L30, SW6 L40, SW7 L01, SW8 L11, SW9 L21, U1 SRV05-4, U2 PCAL9555AHF, U6 ATmega32U4-AU, U9 TCR2EF33, X2 KC2016K

Commit message: Updating component 3d models
Parts:
- moved J3 4.66 mm to (207.4, 60.1)
Routing:
- net /IO Expander/SCL: track 127.6 -> 133.7 mm
- net /IO Expander/SDA: track 136.9 -> 142.7 mm
Changed lines of the file:
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@@
   (general
     (thickness 1.6)
-    (drawings 43)
-    (tracks 1736)
+    (drawings 45)
+    (tracks 1741)
     (zones 0)
     (modules 96)
@@
       (effects (font (size 1 1) (thickness 0.15)))
     )
-    (fp_arc (start -1.986819 -2.7432) (end -1.986819 -2.947981) (angle -90) (layer Dwgs.User) (width 0.05))
-    (fp_arc (start -1.096381 -2.7432) (end -0.8916 -2.7432) (angle -90) (layer Dwgs.User) (width 0.05))
-    (fp_arc (start 7.006219 -2.7432) (end 7.211 -2.7432) (angle -90) (layer Dwgs.User) (width 0.05))
-    (fp_arc (start 6.115781 -2.7432) (end 6.115781 -2.947981) (angle -90) (layer Dwgs.User) (width 0.05))
     (fp_circle (center 0 -2) (end 0.1 -2) (layer F.SilkS) (width 0.2))
     (fp_line (start -0.889 1.8542) (end 5.911 1.8542) (layer Dwgs.User) (width 0.05))
@@
     (fp_line (start -2.1916 1.8542) (end -2.1916 -2.7432) (layer Dwgs.User) (width 0.05))
     (fp_line (start -1.986819 -2.947981) (end -1.096381 -2.947981) (layer Dwgs.User) (width 0.05))
+    (fp_arc (start -1.986819 -2.7432) (end -1.986819 -2.947981) (angle -90) (layer Dwgs.User) (width 0.05))
+    (fp_arc (start -1.096381 -2.7432) (end -0.8916 -2.7432) (angle -90) (layer Dwgs.User) (width 0.05))
+    (fp_arc (start 7.006219 -2.7432) (end 7.211 -2.7432) (angle -90) (layer Dwgs.User) (width 0.05))
+    (fp_arc (start 6.115781 -2.7432) (end 6.115781 -2.947981) (angle -90) (layer Dwgs.User) (width 0.05))
     (pad 6 smd roundrect (at 5 0) (size 1 2.7) (layers B.Cu B.Adhes B.SilkS) (roundrect_rratio 0.25)
       (net 3 GND))
@@
   )
   (module Connector_PinHeader_2.54mm:PinHeader_1x02_P2.54mm_Vertical (layer F.Cu)
-    (at 211.963 60.833 90)
+    (at 207.3529 60.1472 90)
     (descr "Through hole straight pin header, 1x02, 2.54mm pitch, single row")
     (tags "Through hole pin header THT 1x02 2.54mm single row")
@@
     (pad 1 smd oval (at -2.05 -1.25 45) (size 0.24 0.9) (layers F.Cu F.Paste F.Mask)
       (net 123 "/IO Expander/ROW[0]"))
+    (model "C:/Users/binos/Documents/Projects/PCB/library/mechanical/qfn24-4x4-1.snapshot.1/QFN24(4X4).STEP"
+      (offset (xyz 0 0 1))
+      (scale (xyz 1 1 1))
+      (rotate (xyz 90 0 180))
+    )
   )
   (module resistor_smd:R_0603_1608Metric (layer F.Cu)
@@
   (module custom_footprint_library:KC2016K (layer F.Cu)
     (at 123.1028 60.9188 180)
-    (fp_text reference X2 (at 0.4716 1.8892) (layer F.SilkS)
+    (fp_text reference X2 (at 0.3954 2.4099) (layer F.SilkS)
       (effects (font (size 1 1) (thickness 0.15)))
     )
@@
       (net 4 +3V3))
   )
+  (gr_circle (center 153.5176 63.9064) (end 153.6176 63.9064) (layer B.SilkS) (width 0.2))
+  (gr_circle (center 122.19178 59.43346) (end 122.29178 59.43346) (layer F.SilkS) (width 0.2))
   (gr_line (start 105.9815 59.4868) (end 105.1814 59.4868) (layer Edge.Cuts) (width 0.05))
   (gr_line (start 106.23 53.6702) (end 106.2355 59.2328) (layer Edge.Cuts) (width 0.05))
@@
   (segment (start 163.324822 71.374) (end 163.9488 70.750022) (width 0.25) (layer F.Cu) (net 135))
   (segment (start 158.115 71.374) (end 158.223467 71.265533) (width 0.25) (layer F.Cu) (net 135))
-  (segment (start 215.646251 61.976251) (end 214.503 60.833) (width 0.25) (layer F.Cu) (net 135))
   (segment (start 215.646251 66.769999) (end 215.646251 61.976251) (width 0.25) (layer F.Cu) (net 135))
   (segment (start 214.47125 67.945) (end 215.646251 66.769999) (width 0.25) (layer F.Cu) (net 135))
+  (segment (start 213.8172 60.1472) (end 215.4047 61.7347) (width 0.25) (layer F.Cu) (net 135))
+  (segment (start 209.8929 60.1472) (end 213.8172 60.1472) (width 0.25) (layer F.Cu) (net 135))
+  (segment (start 215.4047 61.7347) (end 214.503 60.833) (width 0.25) (layer F.Cu) (net 135))
+  (segment (start 215.646251 61.976251) (end 215.4047 61.7347) (width 0.25) (layer F.Cu) (net 135))
   (segment (start 124.63212 63.826662) (end 124.63212 63.86262) (width 0.25) (layer F.Cu) (net 136))
   (via (at 128.3716 70.04812) (size 0.8) (drill 0.4) (layers F.Cu B.Cu) (net 136))
@@
   (segment (start 211.93125 67.945) (end 213.296249 69.309999) (width 0.25) (layer F.Cu) (net 136))
   (segment (start 215.728801 69.309999) (end 216.4588 68.58) (width 0.25) (layer F.Cu) (net 136))
-  (segment (start 213.138001 59.657999) (end 211.963 60.833) (width 0.25) (layer F.Cu) (net 136))
-  (segment (start 215.067001 59.657999) (end 213.138001 59.657999) (width 0.25) (layer F.Cu) (net 136))
-  (segment (start 216.4588 61.049798) (end 215.067001 59.657999) (width 0.25) (layer F.Cu) (net 136))
-  (segment (start 216.4588 68.58) (end 216.4588 61.049798) (width 0.25) (layer F.Cu) (net 136))
+  (segment (start 216.4588 63.1444) (end 216.4588 60.8965) (width 0.25) (layer F.Cu) (net 136))
+  (segment (start 216.4588 68.58) (end 216.4588 63.1444) (width 0.25) (layer F.Cu) (net 136))
+  (segment (start 216.4588 63.1444) (end 216.4588 62.357) (width 0.25) (layer F.Cu) (net 136))
+  (segment (start 208.527901 58.972199) (end 207.3529 60.1472) (width 0.25) (layer F.Cu) (net 136))
+  (segment (start 214.534499 58.972199) (end 208.527901 58.972199) (width 0.25) (layer F.Cu) (net 136))
+  (segment (start 216.4588 60.8965) (end 214.534499 58.972199) (width 0.25) (layer F.Cu) (net 136))
   (segment (start 211.93125 73.025) (end 211.93125 74.99985) (width 0.25) (layer B.Cu) (net 140))
   (segment (start 215.32126 78.38986) (end 215.32126 83.09631) (width 0.25) (layer B.Cu) (net 140))
