File: Hardware/v0/ergonomic_split_left/uController.sch (KiCad schematic (older format))
At the start: 15 parts, among them J3 Conn_02x03_Odd_Even, SW1 SW_Push, U5 ATmega32U4-AU, X2 KC2016K

Commit message: Connecting schematic blocks, most sub-blocks done
Parts:
- added R14, R15: 2K2, resistor_smd:R_0603_1608Metric, symbol Device:R
Connections:
- net nCAPS is gone; now on net nCAPS_LED: R3.1
- net +3V3: now also R14.1, R15.1
- net SCL: now also R14.2
- net SDA: now also R15.2
- net nCAPS_LED: now reaches U5.22 (PD5)
- net ENCODER_A_L: now reaches U5.26 (PD6)
- net ENCODER_B_L: now reaches U5.27 (PD7)
- net ENCODER_B_R: now reaches U5.38 (PF5)
- net ENCODER_A_R: now reaches U5.39 (PF4)
- net USB_IN+ renamed USB+
- net USB_IN- renamed USB-
Changed lines of the file:
@@
 $Descr A4 11693 8268
 encoding utf-8
-Sheet 3 7
+Sheet 5 7
 Title "TKL Keyboard"
 Date ""
@@
 Wire Wire Line
 	4175 4400 4175 4350
-$Comp
-L Device:R R?
-U 1 1 60D6927E
-P 4175 2400
-AR Path="/60D6927E" Ref="R?"  Part="1"
-AR Path="/60D44BDB/60D6927E" Ref="R?"  Part="1"
-AR Path="/62022D96/60D6927E" Ref="R18"  Part="1"
-AR Path="/612342D1/60D6927E" Ref="R18"  Part="1"
-AR Path="/63013830/60D6927E" Ref="R22"  Part="1"
-AR Path="/62999575/60D6927E" Ref="R22"  Part="1"
-F 0 "R22" H 3975 2475 50  0000 L CNN
-F 1 "10K" V 4175 2350 50  0000 L CNN
-F 2 "resistor_smd:R_0603_1608Metric" V 4105 2400 50  0001 C CNN
-F 3 "~" H 4175 2400 50  0001 C CNN
-	1    4175 2400
-	1    0    0    -1
-$EndComp
 Wire Wire Line
 	4175 2550 4175 2625
@@
 Wire Wire Line
 	3625 2825 4375 2825
-Text GLabel 7975 3475 2    50   Input ~ 0
-MOSI
 $Comp
 L power:GND #PWR?
@@
 	1    0    0    -1
 $EndComp
-Text GLabel 5925 2925 2    50   Output ~ 0
-MISO
-Text GLabel 5925 2725 2    50   Input ~ 0
-SCK
-Text GLabel 5925 2825 2    50   Input ~ 0
-MOSI
 Wire Wire Line
 	5925 2725 5575 2725
 Wire Wire Line
 	5575 2825 5925 2825
-Text GLabel 4100 2625 0    50   Input ~ 0
-RST
 Wire Wire Line
 	4100 2625 4175 2625
@@
 Wire Wire Line
 	6975 3575 7150 3575
-Text GLabel 6975 3575 0    50   Input ~ 0
-RST
-Text GLabel 6975 3475 0    50   Input ~ 0
-SCK
-Text GLabel 6975 3375 0    50   Output ~ 0
-MISO
 $Comp
 L Connector_Generic:Conn_02x03_Odd_Even J?
@@
 	6650 2900 8300 2900
 Text HLabel 3500 3625 0    50   BiDi ~ 0
-USB_IN+
+USB+
 Text HLabel 3500 3725 0    50   BiDi ~ 0
-USB_IN-
+USB-
 Text HLabel 5925 3825 2    50   BiDi ~ 0
 SCL
@@
 Wire Wire Line
 	7675 4825 7675 4875
-Wire Wire Line
-	9375 5750 9025 5750
-Text GLabel 9375 5750 2    50   Input ~ 0
-nCAPS
 $Comp
 L Device:R R?
@@
 Wire Wire Line
 	2500 5475 2500 5525
-Text GLabel 2675 5900 2    50   Input ~ 0
-nCAPS
 Wire Wire Line
 	2500 5900 2500 5825
@@
 Wire Wire Line
 	3500 3625 4375 3625
+$Comp
+L Device:R R?
+U 1 1 60D6927E
+P 4175 2400
+AR Path="/60D6927E" Ref="R?"  Part="1"
+AR Path="/60D44BDB/60D6927E" Ref="R?"  Part="1"
+AR Path="/62022D96/60D6927E" Ref="R18"  Part="1"
+AR Path="/612342D1/60D6927E" Ref="R18"  Part="1"
+AR Path="/63013830/60D6927E" Ref="R22"  Part="1"
+AR Path="/62999575/60D6927E" Ref="R22"  Part="1"
+F 0 "R22" H 3975 2475 50  0000 L CNN
+F 1 "10K" V 4175 2350 50  0000 L CNN
+F 2 "resistor_smd:R_0603_1608Metric" V 4105 2400 50  0001 C CNN
+F 3 "~" H 4175 2400 50  0001 C CNN
+	1    4175 2400
+	1    0    0    -1
+$EndComp
+Text HLabel 5925 4425 2    50   Input ~ 0
+ENCODER_A_L
+Text HLabel 5925 4525 2    50   Input ~ 0
+ENCODER_B_L
+Text HLabel 5925 5225 2    50   Input ~ 0
+ENCODER_A_R
+Text HLabel 5925 5325 2    50   Input ~ 0
+ENCODER_B_R
+Text Label 5925 2725 0    50   ~ 0
+SCK
+Text Label 6975 3475 2    50   ~ 0
+SCK
+Text Label 5925 2825 0    50   ~ 0
+MOSI
+Text Label 7975 3475 0    50   ~ 0
+MOSI
+Text Label 5925 2925 0    50   ~ 0
+MISO
+Text Label 6975 3375 2    50   ~ 0
+MISO
+Text Label 4100 2625 2    50   ~ 0
+RST
+Text Label 6975 3575 2    50   ~ 0
+RST
+Text Label 5925 4325 0    50   ~ 0
+nCAPS_LED
+Text Label 2675 5900 0    50   ~ 0
+nCAPS_LED
+Wire Notes Line
+	8300 6150 8300 5275
+Wire Notes Line
+	8300 5275 6650 5275
+Wire Notes Line
+	6650 5275 6650 6150
+Wire Notes Line
+	6650 6150 8300 6150
+Text HLabel 7250 5675 0    50   BiDi ~ 0
+SCL
+Text HLabel 7250 5775 0    50   BiDi ~ 0
+SDA
+$Comp
+L Device:R R?
+U 1 1 6EAA3992
+P 7550 5675
+AR Path="/6EAA3992" Ref="R?"  Part="1"
+AR Path="/60D44BDB/6EAA3992" Ref="R?"  Part="1"
+AR Path="/62022D96/6EAA3992" Ref="R?"  Part="1"
+AR Path="/612342D1/6EAA3992" Ref="R?"  Part="1"
+AR Path="/63013830/6EAA3992" Ref="R?"  Part="1"
+AR Path="/62999575/6EAA3992" Ref="R14"  Part="1"
+F 0 "R14" V 7550 6000 50  0000 C CNN
+F 1 "2K2" V 7550 5675 50  0000 C CNN
+F 2 "resistor_smd:R_0603_1608Metric" V 7480 5675 50  0001 C CNN
+F 3 "~" H 7550 5675 50  0001 C CNN
+	1    7550 5675
+	0    1    -1   0
+$EndComp
+$Comp
+L Device:R R?
+U 1 1 6EAA6F53
+P 7550 5775
+AR Path="/6EAA6F53" Ref="R?"  Part="1"
+AR Path="/60D44BDB/6EAA6F53" Ref="R?"  Part="1"
+AR Path="/62022D96/6EAA6F53" Ref="R?"  Part="1"
+AR Path="/612342D1/6EAA6F53" Ref="R?"  Part="1"
+AR Path="/63013830/6EAA6F53" Ref="R?"  Part="1"
+AR Path="/62999575/6EAA6F53" Ref="R15"  Part="1"
+F 0 "R15" V 7550 6100 50  0000 C CNN
+F 1 "2K2" V 7550 5775 50  0000 C CNN
+F 2 "resistor_smd:R_0603_1608Metric" V 7480 5775 50  0001 C CNN
+F 3 "~" H 7550 5775 50  0001 C CNN
+	1    7550 5775
+	0    1    -1   0
+$EndComp
+Wire Wire Line
+	7400 5675 7250 5675
+Wire Wire Line
+	7250 5775 7400 5775
+$Comp
+L power:+3.3V #PWR?
+U 1 1 6EAA9FB3
+P 7775 5600
+AR Path="/6EAA9FB3" Ref="#PWR?"  Part="1"
+AR Path="/60D44BDB/6EAA9FB3" Ref="#PWR?"  Part="1"
+AR Path="/62022D96/6EAA9FB3" Ref="#PWR?"  Part="1"
+AR Path="/612342D1/6EAA9FB3" Ref="#PWR?"  Part="1"
+AR Path="/63013830/6EAA9FB3" Ref="#PWR?"  Part="1"
+AR Path="/62999575/6EAA9FB3" Ref="#PWR0203"  Part="1"
+F 0 "#PWR0203" H 7775 5450 50  0001 C CNN
+F 1 "+3.3V" H 7790 5773 50  0000 C CNN
+F 2 "" H 7775 5600 50  0001 C CNN
+F 3 "" H 7775 5600 50  0001 C CNN
+	1    7775 5600
+	1    0    0    -1
+$EndComp
+Wire Wire Line
+	7700 5775 7775 5775
+Wire Wire Line
+	7775 5775 7775 5675
+Wire Wire Line
+	7700 5675 7775 5675
+Connection ~ 7775 5675
+Wire Wire Line
+	7775 5675 7775 5600
+Wire Wire Line
+	5925 5225 5575 5225
+Wire Wire Line
+	5925 5325 5575 5325
+Wire Wire Line
+	5925 4425 5575 4425
+Wire Wire Line
+	5925 4525 5575 4525
+Wire Wire Line
+	5925 4325 5575 4325
 $EndSCHEMATC

Commit message: Adding power and ground planes Adding right interface USB C connector Pin swapping on ATMEGA
Connections:
- net ENCODER_A_L: now also U5.39 (PF4); no longer U5.26 (PD6)
- net ENCODER_A_R: now also U5.41 (PF0); no longer U5.39 (PF4)
- net ENCODER_B_L: now also U5.38 (PF5); no longer U5.27 (PD7)
- net ENCODER_B_R: now also U5.40 (PF1); no longer U5.38 (PF5)
- net nCAPS_LED: now also U5.12 (PB7); no longer U5.22 (PD5)
Changed lines of the file:
@@
 L power:GND #PWR?
 U 1 1 6202CCD8
-P 6425 4800
+P 6025 4775
 AR Path="/6202CCD8" Ref="#PWR?"  Part="1"
 AR Path="/60D44BDB/6202CCD8" Ref="#PWR?"  Part="1"
@@
 AR Path="/63013830/6202CCD8" Ref="#PWR0181"  Part="1"
 AR Path="/62999575/6202CCD8" Ref="#PWR0181"  Part="1"
-F 0 "#PWR0181" H 6425 4550 50  0001 C CNN
-F 1 "GND" H 6430 4627 50  0000 C CNN
-F 2 "" H 6425 4800 50  0001 C CNN
-F 3 "" H 6425 4800 50  0001 C CNN
-	1    6425 4800
-	1    0    0    -1
-$EndComp
-Wire Wire Line
-	5975 4725 6425 4725
-Wire Wire Line
-	6425 4725 6425 4800
+F 0 "#PWR0181" H 6025 4525 50  0001 C CNN
+F 1 "GND" H 6030 4602 50  0000 C CNN
+F 2 "" H 6025 4775 50  0001 C CNN
+F 3 "" H 6025 4775 50  0001 C CNN
+	1    6025 4775
+	1    0    0    -1
+$EndComp
 Wire Wire Line
 	5925 3225 5575 3225
@@
 	1    0    0    -1
 $EndComp
-Text HLabel 5925 4425 2    50   Input ~ 0
+Text HLabel 5925 5225 2    50   Input ~ 0
 ENCODER_A_L
-Text HLabel 5925 4525 2    50   Input ~ 0
+Text HLabel 5925 5325 2    50   Input ~ 0
 ENCODER_B_L
-Text HLabel 5925 5225 2    50   Input ~ 0
+Text HLabel 5925 5025 2    50   Input ~ 0
 ENCODER_A_R
-Text HLabel 5925 5325 2    50   Input ~ 0
+Text HLabel 5925 5125 2    50   Input ~ 0
 ENCODER_B_R
 Text Label 5925 2725 0    50   ~ 0
@@
 Text Label 6975 3575 2    50   ~ 0
 RST
-Text Label 5925 4325 0    50   ~ 0
+Text Label 5925 3325 0    50   ~ 0
 nCAPS_LED
 Text Label 2675 5900 0    50   ~ 0
@@
 	7775 5675 7775 5600
 Wire Wire Line
+	5925 5025 5575 5025
+Wire Wire Line
+	5925 5125 5575 5125
+Wire Wire Line
 	5925 5225 5575 5225
 Wire Wire Line
 	5925 5325 5575 5325
 Wire Wire Line
-	5925 4425 5575 4425
-Wire Wire Line
-	5925 4525 5575 4525
-Wire Wire Line
-	5925 4325 5575 4325
+	5925 3325 5575 3325
+Wire Wire Line
+	6025 4775 6025 4725
+Wire Wire Line
+	6025 4725 5975 4725
 $EndSCHEMATC

Commit message: Debug connectors Adding I2C debug header Changed SPI programming header to edge mount Changed right interface connector to IDC Cleaning up schematic
Parts:
- added J3: Conn_01x02_Male, Connector_PinHeader_2.54mm:PinHeader_1x02_P2.54mm_Vertical, symbol Connector:Conn_01x02_Male
- J3: footprint custom_footprint_library:ISP_POGO -> custom_footprint_library:Conn_AVX_PCB_Edge_02x03
Connections:
- net SCL: now also J3.2 (Pin_2)
- net SDA: now also J3.1 (Pin_1)
Other:
- note added: "I2C"
- moved on the sheet: R14, R15
Changed lines of the file:
@@
 F 0 "J5" H 7400 3775 50  0000 C CNN
 F 1 "Conn_02x03_Odd_Even" H 7175 3700 50  0000 C CNN
-F 2 "custom_footprint_library:ISP_POGO" H 7425 3475 50  0001 C CNN
+F 2 "custom_footprint_library:Conn_AVX_PCB_Edge_02x03" H 7425 3475 50  0001 C CNN
 F 3 "~" H 7425 3475 50  0001 C CNN
 	1    7425 3475
@@
 Wire Notes Line
 	6650 6150 8300 6150
-Text HLabel 7250 5675 0    50   BiDi ~ 0
+Text HLabel 6900 5950 0    50   BiDi ~ 0
 SCL
-Text HLabel 7250 5775 0    50   BiDi ~ 0
+Text HLabel 6900 6050 0    50   BiDi ~ 0
 SDA
 $Comp
 L Device:R R?
 U 1 1 6EAA3992
-P 7550 5675
+P 7375 5725
 AR Path="/6EAA3992" Ref="R?"  Part="1"
 AR Path="/60D44BDB/6EAA3992" Ref="R?"  Part="1"
@@
 AR Path="/63013830/6EAA3992" Ref="R?"  Part="1"
 AR Path="/62999575/6EAA3992" Ref="R14"  Part="1"
-F 0 "R14" V 7550 6000 50  0000 C CNN
-F 1 "2K2" V 7550 5675 50  0000 C CNN
-F 2 "resistor_smd:R_0603_1608Metric" V 7480 5675 50  0001 C CNN
-F 3 "~" H 7550 5675 50  0001 C CNN
-	1    7550 5675
-	0    1    -1   0
+F 0 "R14" H 7500 5750 50  0000 C CNN
+F 1 "2K2" V 7375 5725 50  0000 C CNN
+F 2 "resistor_smd:R_0603_1608Metric" V 7305 5725 50  0001 C CNN
+F 3 "~" H 7375 5725 50  0001 C CNN
+	1    7375 5725
+	-1   0    0    -1
 $EndComp
 $Comp
 L Device:R R?
 U 1 1 6EAA6F53
-P 7550 5775
+P 7475 5725
 AR Path="/6EAA6F53" Ref="R?"  Part="1"
 AR Path="/60D44BDB/6EAA6F53" Ref="R?"  Part="1"
@@
 AR Path="/63013830/6EAA6F53" Ref="R?"  Part="1"
 AR Path="/62999575/6EAA6F53" Ref="R15"  Part="1"
-F 0 "R15" V 7550 6100 50  0000 C CNN
-F 1 "2K2" V 7550 5775 50  0000 C CNN
-F 2 "resistor_smd:R_0603_1608Metric" V 7480 5775 50  0001 C CNN
-F 3 "~" H 7550 5775 50  0001 C CNN
-	1    7550 5775
-	0    1    -1   0
-$EndComp
-Wire Wire Line
-	7400 5675 7250 5675
-Wire Wire Line
-	7250 5775 7400 5775
+F 0 "R15" H 7350 5750 50  0000 C CNN
+F 1 "2K2" V 7475 5725 50  0000 C CNN
+F 2 "resistor_smd:R_0603_1608Metric" V 7405 5725 50  0001 C CNN
+F 3 "~" H 7475 5725 50  0001 C CNN
+	1    7475 5725
+	-1   0    0    -1
+$EndComp
 $Comp
 L power:+3.3V #PWR?
 U 1 1 6EAA9FB3
-P 7775 5600
+P 7375 5475
 AR Path="/6EAA9FB3" Ref="#PWR?"  Part="1"
 AR Path="/60D44BDB/6EAA9FB3" Ref="#PWR?"  Part="1"
@@
 AR Path="/63013830/6EAA9FB3" Ref="#PWR?"  Part="1"
 AR Path="/62999575/6EAA9FB3" Ref="#PWR0203"  Part="1"
-F 0 "#PWR0203" H 7775 5450 50  0001 C CNN
-F 1 "+3.3V" H 7790 5773 50  0000 C CNN
-F 2 "" H 7775 5600 50  0001 C CNN
-F 3 "" H 7775 5600 50  0001 C CNN
-	1    7775 5600
-	1    0    0    -1
-$EndComp
-Wire Wire Line
-	7700 5775 7775 5775
-Wire Wire Line
-	7775 5775 7775 5675
-Wire Wire Line
-	7700 5675 7775 5675
-Connection ~ 7775 5675
-Wire Wire Line
-	7775 5675 7775 5600
+F 0 "#PWR0203" H 7375 5325 50  0001 C CNN
+F 1 "+3.3V" H 7375 5625 50  0000 C CNN
+F 2 "" H 7375 5475 50  0001 C CNN
+F 3 "" H 7375 5475 50  0001 C CNN
+	1    7375 5475
+	1    0    0    -1
+$EndComp
 Wire Wire Line
 	5925 5025 5575 5025
@@
 Wire Wire Line
 	6025 4725 5975 4725
+$Comp
+L Connector:Conn_01x02_Male J3
+U 1 1 62DE68FB
+P 7800 6050
+F 0 "J3" H 7772 5932 50  0000 R CNN
+F 1 "Conn_01x02_Male" H 8000 6100 50  0000 R CNN
+F 2 "Connector_PinHeader_2.54mm:PinHeader_1x02_P2.54mm_Vertical" H 7800 6050 50  0001 C CNN
+F 3 "~" H 7800 6050 50  0001 C CNN
+	1    7800 6050
+	-1   0    0    1
+$EndComp
+Wire Wire Line
+	7375 5475 7375 5525
+Wire Wire Line
+	7475 5575 7475 5525
+Wire Wire Line
+	7475 5525 7375 5525
+Connection ~ 7375 5525
+Wire Wire Line
+	7375 5525 7375 5575
+Wire Wire Line
+	7375 5950 7375 5875
+Wire Wire Line
+	6900 5950 7375 5950
+Wire Wire Line
+	7475 6050 7475 5875
+Wire Wire Line
+	6900 6050 7475 6050
+Wire Wire Line
+	7600 5950 7375 5950
+Connection ~ 7375 5950
+Wire Wire Line
+	7600 6050 7475 6050
+Connection ~ 7475 6050
+Text Notes 6700 5375 0    50   ~ 0
+I2C
 $EndSCHEMATC

Commit message: Prelim routing done
Connections:
- net ENCODER_A_L: now also U5.40 (PF1); no longer U5.39 (PF4)
- net ENCODER_A_R: now also U5.39 (PF4); no longer U5.41 (PF0)
- net ENCODER_B_L: now also U5.41 (PF0); no longer U5.38 (PF5)
- net ENCODER_B_R: now also U5.38 (PF5); no longer U5.40 (PF1)
Changed lines of the file:
@@
 	1    0    0    -1
 $EndComp
+Text HLabel 5925 5125 2    50   Input ~ 0
+ENCODER_A_L
+Text HLabel 5925 5025 2    50   Input ~ 0
+ENCODER_B_L
 Text HLabel 5925 5225 2    50   Input ~ 0
-ENCODER_A_L
+ENCODER_A_R
 Text HLabel 5925 5325 2    50   Input ~ 0
-ENCODER_B_L
-Text HLabel 5925 5025 2    50   Input ~ 0
-ENCODER_A_R
-Text HLabel 5925 5125 2    50   Input ~ 0
 ENCODER_B_R
 Text Label 5925 2725 0    50   ~ 0

Commit message: Cleaning up routing
Connections:
- net nCAPS_LED: now also U5.1 (PE6); no longer U5.12 (PB7)
Changed lines of the file:
@@
 L power:GND #PWR?
 U 1 1 6202CCD8
-P 6025 4775
+P 6450 4775
 AR Path="/6202CCD8" Ref="#PWR?"  Part="1"
 AR Path="/60D44BDB/6202CCD8" Ref="#PWR?"  Part="1"
@@
 AR Path="/63013830/6202CCD8" Ref="#PWR0181"  Part="1"
 AR Path="/62999575/6202CCD8" Ref="#PWR0181"  Part="1"
-F 0 "#PWR0181" H 6025 4525 50  0001 C CNN
-F 1 "GND" H 6030 4602 50  0000 C CNN
-F 2 "" H 6025 4775 50  0001 C CNN
-F 3 "" H 6025 4775 50  0001 C CNN
-	1    6025 4775
+F 0 "#PWR0181" H 6450 4525 50  0001 C CNN
+F 1 "GND" H 6455 4602 50  0000 C CNN
+F 2 "" H 6450 4775 50  0001 C CNN
+F 3 "" H 6450 4775 50  0001 C CNN
+	1    6450 4775
 	1    0    0    -1
 $EndComp
@@
 Text Label 6975 3575 2    50   ~ 0
 RST
-Text Label 5925 3325 0    50   ~ 0
+Text Label 5925 4825 0    50   ~ 0
 nCAPS_LED
 Text Label 2675 5900 0    50   ~ 0
@@
 	5925 5325 5575 5325
 Wire Wire Line
-	5925 3325 5575 3325
-Wire Wire Line
-	6025 4775 6025 4725
-Wire Wire Line
-	6025 4725 5975 4725
+	5925 4825 5575 4825
 $Comp
 L Connector:Conn_01x02_Male J3
@@
 Text Notes 6700 5375 0    50   ~ 0
 I2C
+Wire Wire Line
+	5975 4725 6450 4725
+Wire Wire Line
+	6450 4725 6450 4775
 $EndSCHEMATC
